Commit message: Add range data to gridmap Update raytracing for speed

File: gridmap/test/robot.urdf.xacro (robot description, xacro)
@@ -68,5 +68,5 @@
         <sensor type="ray" name="laser">
             <pose>0 0 0 0 0 0</pose>
-            <visualize>false</visualize>
+            <visualize>true</visualize>
             <update_rate>40</update_rate>
             <ray>
@@ -96,3 +96,77 @@
         </sensor>
     </gazebo>
+    <xacro:macro name="range_sensor" params="suffix rotation">
+        <joint name="range_${suffix}_joint" type="fixed">
+            <origin xyz="0 0 0.4" rpy="0 0 ${rotation}"/>
+            <child link="range_${suffix}"/>
+            <parent link="base_link"/>
+        </joint>
+        <link name="range_${suffix}">
+            <visual>
+                <origin xyz="0 0 0"/>
+                <geometry>
+                    <cylinder length="0.05" radius="0.05"/>
+                </geometry>
+            </visual>
+            <collision>
+                <origin xyz="0 0 0"/>
+                <geometry>
+                    <cylinder length="0.05" radius="0.05"/>
+                </geometry>
+            </collision>
+            <inertial>
+                <mass value="1"/>
+                <origin xyz="0 0 0"/>
+                <inertia
+                        ixx="1" ixy="0" ixz="0"
+                        iyy="1" iyz="0"
+                        izz="1"/>
+            </inertial>
+        </link>
+        <gazebo reference="range_${suffix}">
+            <sensor type="ray" name="range_${suffix}">
+                <pose>0 0 0 0 0 0</pose>
+                <visualize>true</visualize>
+                <update_rate>10</update_rate>
+                <ray>
+                    <scan>
+                        <horizontal>
+                            <samples>10</samples>
+                            <resolution>1</resolution>
+                            <min_angle>-0.4</min_angle>
+                            <max_angle>0.4</max_angle>
+                        </horizontal>
+                        <vertical>
+                            <samples>10</samples>
+                            <resolution>1</resolution>
+                            <min_angle>-0.2</min_angle>
+                            <max_angle>0.2</max_angle>
+                        </vertical>
+                    </scan>
+                    <range>
+                        <min>0.1</min>
+                        <max>2.0</max>
+                        <resolution>0.01</resolution>
+                    </range>
+                </ray>
+                <plugin name="gazebo_range_plugin" filename="libgazebo_range_plugin.so">
+                    <robot_namespace>/</robot_namespace>
+                    <field_of_view>0.8</field_of_view>
+                </plugin>
+            </sensor>
+        </gazebo>
+    </xacro:macro>
+    <xacro:range_sensor suffix="0" rotation="-3.0"/>
+    <xacro:range_sensor suffix="1" rotation="-2.5"/>
+    <xacro:range_sensor suffix="2" rotation="-2.0"/>
+    <xacro:range_sensor suffix="3" rotation="-1.5"/>
+    <xacro:range_sensor suffix="4" rotation="-1.0"/>
+    <xacro:range_sensor suffix="5" rotation="-0.5"/>
+    <xacro:range_sensor suffix="6" rotation="0.0"/>
+    <xacro:range_sensor suffix="7" rotation="0.5"/>
+    <xacro:range_sensor suffix="8" rotation="1.0"/>
+    <xacro:range_sensor suffix="9" rotation="1.5"/>
+    <xacro:range_sensor suffix="10" rotation="2.0"/>
+    <xacro:range_sensor suffix="11" rotation="2.5"/>
+    <xacro:range_sensor suffix="12" rotation="3.0"/>
 </robot>

Commit message: Update sonar sensor model to fast rasterize a triangle Fix astar to add goal pose Fix yaw calculation in move_base Fix yaw calculation in pure_pursuit_controller

File: gridmap/test/robot.urdf.xacro (robot description, xacro)
@@ -96,11 +96,11 @@
         </sensor>
     </gazebo>
-    <xacro:macro name="range_sensor" params="suffix rotation">
-        <joint name="range_${suffix}_joint" type="fixed">
+    <xacro:macro name="sonar_sensor" params="suffix rotation">
+        <joint name="sonar_${suffix}_joint" type="fixed">
             <origin xyz="0 0 0.4" rpy="0 0 ${rotation}"/>
-            <child link="range_${suffix}"/>
+            <child link="sonar_${suffix}"/>
             <parent link="base_link"/>
         </joint>
-        <link name="range_${suffix}">
+        <link name="sonar_${suffix}">
             <visual>
                 <origin xyz="0 0 0"/>
@@ -124,6 +124,6 @@
             </inertial>
         </link>
-        <gazebo reference="range_${suffix}">
-            <sensor type="ray" name="range_${suffix}">
+        <gazebo reference="sonar_${suffix}">
+            <sensor type="ray" name="sonar_${suffix}">
                 <pose>0 0 0 0 0 0</pose>
                 <visualize>true</visualize>
@@ -145,6 +145,6 @@
                     </scan>
                     <range>
-                        <min>0.1</min>
-                        <max>2.0</max>
+                        <min>0.15</min>
+                        <max>1.5</max>
                         <resolution>0.01</resolution>
                     </range>
@@ -157,16 +157,16 @@
         </gazebo>
     </xacro:macro>
-    <xacro:range_sensor suffix="0" rotation="-3.0"/>
-    <xacro:range_sensor suffix="1" rotation="-2.5"/>
-    <xacro:range_sensor suffix="2" rotation="-2.0"/>
-    <xacro:range_sensor suffix="3" rotation="-1.5"/>
-    <xacro:range_sensor suffix="4" rotation="-1.0"/>
-    <xacro:range_sensor suffix="5" rotation="-0.5"/>
-    <xacro:range_sensor suffix="6" rotation="0.0"/>
-    <xacro:range_sensor suffix="7" rotation="0.5"/>
-    <xacro:range_sensor suffix="8" rotation="1.0"/>
-    <xacro:range_sensor suffix="9" rotation="1.5"/>
-    <xacro:range_sensor suffix="10" rotation="2.0"/>
-    <xacro:range_sensor suffix="11" rotation="2.5"/>
-    <xacro:range_sensor suffix="12" rotation="3.0"/>
+    <xacro:sonar_sensor suffix="0" rotation="-3.0"/>
+    <xacro:sonar_sensor suffix="1" rotation="-2.5"/>
+    <xacro:sonar_sensor suffix="2" rotation="-2.0"/>
+    <xacro:sonar_sensor suffix="3" rotation="-1.5"/>
+    <xacro:sonar_sensor suffix="4" rotation="-1.0"/>
+    <xacro:sonar_sensor suffix="5" rotation="-0.5"/>
+    <xacro:sonar_sensor suffix="6" rotation="0.0"/>
+    <xacro:sonar_sensor suffix="7" rotation="0.5"/>
+    <xacro:sonar_sensor suffix="8" rotation="1.0"/>
+    <xacro:sonar_sensor suffix="9" rotation="1.5"/>
+    <xacro:sonar_sensor suffix="10" rotation="2.0"/>
+    <xacro:sonar_sensor suffix="11" rotation="2.5"/>
+    <xacro:sonar_sensor suffix="12" rotation="3.0"/>
 </robot>

Commit message: Update map_manager schema

File: gridmap/test/robot.urdf.xacro (robot description, xacro)
@@ -38,4 +38,13 @@
         </inertial>
     </link>
+    <gazebo reference="base_link">
+        <mu1>0.0</mu1>
+        <mu2>0.0</mu2>
+        <maxVel>0.0</maxVel>
+        <minDepth>0.001</minDepth>
+        <kp>1000000.0</kp>
+        <kd>1.0</kd>
+        <material>Gazebo/Black</material>
+    </gazebo>
     <joint name="laser_joint" type="fixed">
         <origin xyz="0 0 0.2"/>
@@ -69,5 +78,5 @@
             <pose>0 0 0 0 0 0</pose>
             <visualize>true</visualize>
-            <update_rate>40</update_rate>
+            <update_rate>0</update_rate>
             <ray>
                 <scan>
@@ -75,6 +84,6 @@
                         <samples>540</samples>
                         <resolution>1</resolution>
-                        <min_angle>-2.35619</min_angle>
-                        <max_angle>2.35619</max_angle>
+                        <min_angle>-2</min_angle>
+                        <max_angle>2</max_angle>
                     </horizontal>
                 </scan>
@@ -84,9 +93,9 @@
                     <resolution>0.01</resolution>
                 </range>
-                <noise>
-                    <type>gaussian</type>
-                    <mean>0.0</mean>
-                    <stddev>0.001</stddev>
-                </noise>
+                <!--<noise>-->
+                    <!--<type>gaussian</type>-->
+                    <!--<mean>0.0</mean>-->
+                    <!--<stddev>0.001</stddev>-->
+                <!--</noise>-->
             </ray>
             <plugin name="gazebo_laser_plugin" filename="libgazebo_laser_plugin.so">
@@ -157,16 +166,72 @@
         </gazebo>
     </xacro:macro>
-    <xacro:sonar_sensor suffix="0" rotation="-3.0"/>
-    <xacro:sonar_sensor suffix="1" rotation="-2.5"/>
-    <xacro:sonar_sensor suffix="2" rotation="-2.0"/>
-    <xacro:sonar_sensor suffix="3" rotation="-1.5"/>
-    <xacro:sonar_sensor suffix="4" rotation="-1.0"/>
-    <xacro:sonar_sensor suffix="5" rotation="-0.5"/>
-    <xacro:sonar_sensor suffix="6" rotation="0.0"/>
-    <xacro:sonar_sensor suffix="7" rotation="0.5"/>
-    <xacro:sonar_sensor suffix="8" rotation="1.0"/>
-    <xacro:sonar_sensor suffix="9" rotation="1.5"/>
-    <xacro:sonar_sensor suffix="10" rotation="2.0"/>
-    <xacro:sonar_sensor suffix="11" rotation="2.5"/>
-    <xacro:sonar_sensor suffix="12" rotation="3.0"/>
+    <!--<xacro:sonar_sensor suffix="0" rotation="-3.0"/>-->
+    <!--<xacro:sonar_sensor suffix="1" rotation="-2.5"/>-->
+    <!--<xacro:sonar_sensor suffix="2" rotation="-2.0"/>-->
+    <!--<xacro:sonar_sensor suffix="3" rotation="-1.5"/>-->
+    <!--<xacro:sonar_sensor suffix="4" rotation="-1.0"/>-->
+    <!--<xacro:sonar_sensor suffix="5" rotation="-0.5"/>-->
+    <!--<xacro:sonar_sensor suffix="6" rotation="0.0"/>-->
+    <!--<xacro:sonar_sensor suffix="7" rotation="0.5"/>-->
+    <!--<xacro:sonar_sensor suffix="8" rotation="1.0"/>-->
+    <!--<xacro:sonar_sensor suffix="9" rotation="1.5"/>-->
+    <!--<xacro:sonar_sensor suffix="10" rotation="2.0"/>-->
+    <!--<xacro:sonar_sensor suffix="11" rotation="2.5"/>-->
+    <!--<xacro:sonar_sensor suffix="12" rotation="3.0"/>-->
+    <joint name="camera_joint" type="fixed">
+        <origin xyz="0.0 0.0 0.6" rpy="0.0 ${pi/2} 0.0"/>
+        <parent link="base_link"/>
+        <child link="camera"/>
+    </joint>
+    <gazebo reference="camera_joint">
+        <disableFixedJointLumping>true</disableFixedJointLumping>
+    </gazebo>
+    <link name="camera">
+        <inertial>
+            <mass value="1"/>
+            <inertia ixx="1e-6" ixy="0" ixz="0" iyy="1e-6" iyz="0" izz="1e-6"/>
+        </inertial>
+        <visual>
+            <origin xyz="0 0 0.01" rpy="0 0 0"/>
+            <geometry>
+                <cylinder radius="0.016" length="0.080"/>
+            </geometry>
+            <material name="black"/>
+        </visual>
+        <collision>
+            <origin xyz="0 0 0.01" rpy="0 0 0"/>
+            <geometry>
+                <cylinder radius="0.016" length="0.080"/>
+            </geometry>
+        </collision>
+    </link>
+    <gazebo reference="camera">
+        <material>Gazebo/Grey</material>
+        <sensor type="camera" name="camera">
+            <update_rate>1</update_rate>
+            <camera name="camera">
+                <pose>0 0 0 0 ${-pi/2} ${pi/2}</pose>
+                <horizontal_fov>1.5</horizontal_fov>
+                <image>
+                    <width>2560</width>
+                    <height>1920</height>
+                    <format>R8G8B8</format>
+                </image>
+                <clip>
+                    <near>0.01</near>
+                    <far>100</far>
+                </clip>
+                <noise>
+                    <type>gaussian</type>
+                    <mean>0.0</mean>
+                    <stddev>0.00</stddev>
+                </noise>
+            </camera>
+            <plugin name="camera_controller" filename="libgazebo_modular_camera_plugin.so">
+                <camera_name>camera</camera_name>
+                <updateRate>0</updateRate>
+                <frame_name>camera</frame_name>
+            </plugin>
+        </sensor>
+    </gazebo>
 </robot>

Commit message: Update test files Add .rosinstall for `modular_cartographer`

File: gridmap/test/robot.urdf.xacro (robot description, xacro)
@@ -47,62 +47,66 @@
         <material>Gazebo/Black</material>
     </gazebo>
-    <joint name="laser_joint" type="fixed">
-        <origin xyz="0 0 0.2"/>
-        <child link="laser"/>
-        <parent link="base_link"/>
-    </joint>
-    <link name="laser">
-        <visual>
-            <origin xyz="0 0 0"/>
-            <geometry>
-                <cylinder length="0.05" radius="0.05"/>
-            </geometry>
-        </visual>
-        <collision>
-            <origin xyz="0 0 0"/>
-            <geometry>
-                <cylinder length="0.05" radius="0.05"/>
-            </geometry>
-        </collision>
-        <inertial>
-            <mass value="1"/>
-            <origin xyz="0 0 0"/>
-            <inertia
-                    ixx="1" ixy="0" ixz="0"
-                    iyy="1" iyz="0"
-                    izz="1"/>
-        </inertial>
-    </link>
-    <gazebo reference="laser">
-        <sensor type="ray" name="laser">
-            <pose>0 0 0 0 0 0</pose>
-            <visualize>false</visualize>
-            <update_rate>0</update_rate>
-            <ray>
-                <scan>
-                    <horizontal>
-                        <samples>540</samples>
-                        <resolution>1</resolution>
-                        <min_angle>-2</min_angle>
-                        <max_angle>2</max_angle>
-                    </horizontal>
-                </scan>
-                <range>
-                    <min>0.1</min>
-                    <max>30.0</max>
-                    <resolution>0.01</resolution>
-                </range>
-                <!--<noise>-->
-                    <!--<type>gaussian</type>-->
-                    <!--<mean>0.0</mean>-->
-                    <!--<stddev>0.001</stddev>-->
-                <!--</noise>-->
-            </ray>
-            <plugin name="gazebo_laser_plugin" filename="libgazebo_laser_plugin.so">
-                <frame_name>laser</frame_name>
-                <robot_namespace>/</robot_namespace>
-            </plugin>
-        </sensor>
-    </gazebo>
+    <xacro:macro name="laser_sensor" params="suffix rotation">
+        <joint name="laser_joint_${suffix}" type="fixed">
+            <origin xyz="0 0 0.4" rpy="0 0 ${rotation}"/>
+            <child link="laser_${suffix}"/>
+            <parent link="base_link"/>
+        </joint>
+        <link name="laser_${suffix}">
+            <visual>
+                <origin xyz="0 0 0"/>
+                <geometry>
+                    <cylinder length="0.05" radius="0.05"/>
+                </geometry>
+            </visual>
+            <collision>
+                <origin xyz="0 0 0"/>
+                <geometry>
+                    <cylinder length="0.05" radius="0.05"/>
+                </geometry>
+            </collision>
+            <inertial>
+                <mass value="1"/>
+                <origin xyz="0 0 0"/>
+                <inertia
+                        ixx="1" ixy="0" ixz="0"
+                        iyy="1" iyz="0"
+                        izz="1"/>
+            </inertial>
+        </link>
+        <gazebo reference="laser_${suffix}">
+            <sensor type="ray" name="laser_${suffix}">
+                <pose>0 0 0 0 0 0</pose>
+                <visualize>false</visualize>
+                <update_rate>40</update_rate>
+                <ray>
+                    <scan>
+                        <horizontal>
+                            <samples>540</samples>
+                            <resolution>1</resolution>
+                            <min_angle>-2.35619</min_angle>
+                            <max_angle>2.35619</max_angle>
+                        </horizontal>
+                    </scan>
+                    <range>
+                        <min>0.1</min>
+                        <max>30.0</max>
+                        <resolution>0.01</resolution>
+                    </range>
+                    <noise>
+                        <type>gaussian</type>
+                        <mean>0.0</mean>
+                        <stddev>0.001</stddev>
+                    </noise>
+                </ray>
+                <plugin name="gazebo_laser_plugin" filename="libgazebo_laser_plugin.so">
+                    <frame_name>laser_${suffix}</frame_name>
+                    <robot_namespace>/</robot_namespace>
+                </plugin>
+            </sensor>
+        </gazebo>
+    </xacro:macro>
+    <xacro:laser_sensor suffix="front" rotation="0.0"/>
+    <xacro:laser_sensor suffix="back" rotation="${pi}"/>
     <xacro:macro name="sonar_sensor" params="suffix rotation">
         <joint name="sonar_${suffix}_joint" type="fixed">

File: modular_move_base/test/robot.urdf.xacro (robot description, xacro)
@@ -38,62 +38,66 @@
         </inertial>
     </link>
-    <joint name="laser_joint" type="fixed">
-        <origin xyz="0 0 0.2"/>
-        <child link="laser"/>
-        <parent link="base_link"/>
-    </joint>
-    <link name="laser">
-        <visual>
-            <origin xyz="0 0 0"/>
-            <geometry>
-                <cylinder length="0.05" radius="0.05"/>
-            </geometry>
-        </visual>
-        <collision>
-            <origin xyz="0 0 0"/>
-            <geometry>
-                <cylinder length="0.05" radius="0.05"/>
-            </geometry>
-        </collision>
-        <inertial>
-            <mass value="1"/>
-            <origin xyz="0 0 0"/>
-            <inertia
-                    ixx="1" ixy="0" ixz="0"
-                    iyy="1" iyz="0"
-                    izz="1"/>
-        </inertial>
-    </link>
-    <gazebo reference="laser">
-        <sensor type="ray" name="laser">
-            <pose>0 0 0 0 0 0</pose>
-            <visualize>false</visualize>
-            <update_rate>40</update_rate>
-            <ray>
-                <scan>
-                    <horizontal>
-                        <samples>540</samples>
-                        <resolution>1</resolution>
-                        <min_angle>-2.35619</min_angle>
-                        <max_angle>2.35619</max_angle>
-                    </horizontal>
-                </scan>
-                <range>
-                    <min>0.1</min>
-                    <max>30.0</max>
-                    <resolution>0.01</resolution>
-                </range>
-                <noise>
-                    <type>gaussian</type>
-                    <mean>0.0</mean>
-                    <stddev>0.001</stddev>
-                </noise>
-            </ray>
-            <plugin name="gazebo_laser_plugin" filename="libgazebo_laser_plugin.so">
-                <frame_name>laser</frame_name>
-                <robot_namespace>/</robot_namespace>
-            </plugin>
-        </sensor>
-    </gazebo>
+    <xacro:macro name="laser_sensor" params="suffix rotation">
+        <joint name="laser_joint_${suffix}" type="fixed">
+            <origin xyz="0 0 0.4" rpy="0 0 ${rotation}"/>
+            <child link="laser_${suffix}"/>
+            <parent link="base_link"/>
+        </joint>
+        <link name="laser_${suffix}">
+            <visual>
+                <origin xyz="0 0 0"/>
+                <geometry>
+                    <cylinder length="0.05" radius="0.05"/>
+                </geometry>
+            </visual>
+            <collision>
+                <origin xyz="0 0 0"/>
+                <geometry>
+                    <cylinder length="0.05" radius="0.05"/>
+                </geometry>
+            </collision>
+            <inertial>
+                <mass value="1"/>
+                <origin xyz="0 0 0"/>
+                <inertia
+                        ixx="1" ixy="0" ixz="0"
+                        iyy="1" iyz="0"
+                        izz="1"/>
+            </inertial>
+        </link>
+        <gazebo reference="laser_${suffix}">
+            <sensor type="ray" name="laser_${suffix}">
+                <pose>0 0 0 0 0 0</pose>
+                <visualize>false</visualize>
+                <update_rate>40</update_rate>
+                <ray>
+                    <scan>
+                        <horizontal>
+                            <samples>540</samples>
+                            <resolution>1</resolution>
+                            <min_angle>-2.35619</min_angle>
+                            <max_angle>2.35619</max_angle>
+                        </horizontal>
+                    </scan>
+                    <range>
+                        <min>0.1</min>
+                        <max>30.0</max>
+                        <resolution>0.01</resolution>
+                    </range>
+                    <noise>
+                        <type>gaussian</type>
+                        <mean>0.0</mean>
+                        <stddev>0.001</stddev>
+                    </noise>
+                </ray>
+                <plugin name="gazebo_laser_plugin" filename="libgazebo_laser_plugin.so">
+                    <frame_name>laser_${suffix}</frame_name>
+                    <robot_namespace>/</robot_namespace>
+                </plugin>
+            </sensor>
+        </gazebo>
+    </xacro:macro>
+    <xacro:laser_sensor suffix="front" rotation="0.0"/>
+    <xacro:laser_sensor suffix="back" rotation="${pi}"/>
     <xacro:macro name="sonar_sensor" params="suffix rotation">
         <joint name="sonar_${suffix}_joint" type="fixed">
