Commit message: Auto-format with vscode

File: autonomy/test/robot.urdf.xacro (robot description, xacro)
@@ -18,62 +18,62 @@
     <xacro:macro name="robot_circle" params="x_offset y_offset radius">
         <visual>
-            <origin xyz="${x_offset} ${y_offset} 0"/>
+            <origin xyz="${x_offset} ${y_offset} 0" />
             <geometry>
-                <cylinder length="0.05" radius="${radius}"/>
+                <cylinder length="0.05" radius="${radius}" />
             </geometry>
         </visual>
         <collision>
-            <origin xyz="${x_offset} ${y_offset} 0"/>
+            <origin xyz="${x_offset} ${y_offset} 0" />
             <geometry>
-                <cylinder length="0.05" radius="${radius}"/>
+                <cylinder length="0.05" radius="${radius}" />
             </geometry>
         </collision>
     </xacro:macro>
     <link name="base_link">
-        <xacro:robot_circle x_offset="-0.268" y_offset=" 0.000" radius="0.210"/>
-        <xacro:robot_circle x_offset=" 0.268" y_offset=" 0.000" radius="0.210"/>
-        <xacro:robot_circle x_offset=" 0.265" y_offset="-0.185" radius="0.210"/>
-        <xacro:robot_circle x_offset=" 0.077" y_offset="-0.185" radius="0.210"/>
-        <xacro:robot_circle x_offset="-0.077" y_offset="-0.185" radius="0.210"/>
-        <xacro:robot_circle x_offset="-0.265" y_offset="-0.185" radius="0.210"/>
-        <xacro:robot_circle x_offset=" 0.265" y_offset=" 0.185" radius="0.210"/>
-        <xacro:robot_circle x_offset="-0.265" y_offset=" 0.185" radius="0.210"/>
-        <xacro:robot_circle x_offset="-0.077" y_offset=" 0.185" radius="0.210"/>
-        <xacro:robot_circle x_offset=" 0.077" y_offset=" 0.185" radius="0.210"/>
+        <xacro:robot_circle x_offset="-0.268" y_offset=" 0.000" radius="0.210" />
+        <xacro:robot_circle x_offset=" 0.268" y_offset=" 0.000" radius="0.210" />
+        <xacro:robot_circle x_offset=" 0.265" y_offset="-0.185" radius="0.210" />
+        <xacro:robot_circle x_offset=" 0.077" y_offset="-0.185" radius="0.210" />
+        <xacro:robot_circle x_offset="-0.077" y_offset="-0.185" radius="0.210" />
+        <xacro:robot_circle x_offset="-0.265" y_offset="-0.185" radius="0.210" />
+        <xacro:robot_circle x_offset=" 0.265" y_offset=" 0.185" radius="0.210" />
+        <xacro:robot_circle x_offset="-0.265" y_offset=" 0.185" radius="0.210" />
+        <xacro:robot_circle x_offset="-0.077" y_offset=" 0.185" radius="0.210" />
+        <xacro:robot_circle x_offset=" 0.077" y_offset=" 0.185" radius="0.210" />
         <inertial>
-            <origin xyz="0 0 0" rpy="0 0 0"/>
-            <mass value="1"/>
+            <origin xyz="0 0 0" rpy="0 0 0" />
+            <mass value="1" />
             <inertia
-                    ixx="1" ixy="0" ixz="0"
-                    iyy="1" iyz="0"
-                    izz="1"/>
+                ixx="1" ixy="0" ixz="0"
+                iyy="1" iyz="0"
+                izz="1" />
         </inertial>
     </link>
     <xacro:macro name="laser_sensor" params="suffix rotation">
         <joint name="laser_joint_${suffix}" type="fixed">
-            <origin xyz="0 0 0.4" rpy="0 0 ${rotation}"/>
-            <child link="laser_${suffix}"/>
-            <parent link="base_link"/>
+            <origin xyz="0 0 0.4" rpy="0 0 ${rotation}" />
+            <child link="laser_${suffix}" />
+            <parent link="base_link" />
         </joint>
         <link name="laser_${suffix}">
             <visual>
-                <origin xyz="0 0 0"/>
-                <geometry>
-                    <cylinder length="0.05" radius="0.05"/>
+                <origin xyz="0 0 0" />
+                <geometry>
+                    <cylinder length="0.05" radius="0.05" />
                 </geometry>
             </visual>
             <collision>
-                <origin xyz="0 0 0"/>
-                <geometry>
-                    <cylinder length="0.05" radius="0.05"/>
+                <origin xyz="0 0 0" />
+                <geometry>
+                    <cylinder length="0.05" radius="0.05" />
                 </geometry>
             </collision>
             <inertial>
-                <mass value="1"/>
-                <origin xyz="0 0 0"/>
+                <mass value="1" />
+                <origin xyz="0 0 0" />
                 <inertia
-                        ixx="1" ixy="0" ixz="0"
-                        iyy="1" iyz="0"
-                        izz="1"/>
+                    ixx="1" ixy="0" ixz="0"
+                    iyy="1" iyz="0"
+                    izz="1" />
             </inertial>
         </link>
@@ -110,32 +110,32 @@
         </gazebo>
     </xacro:macro>
-    <xacro:laser_sensor suffix="front" rotation="0.0"/>
-    <xacro:laser_sensor suffix="back" rotation="${pi}"/>
+    <xacro:laser_sensor suffix="front" rotation="0.0" />
+    <xacro:laser_sensor suffix="back" rotation="${pi}" />
     <xacro:macro name="sonar_sensor" params="suffix rotation">
         <joint name="sonar_${suffix}_joint" type="fixed">
-            <origin xyz="0 0 0.4" rpy="0 0 ${rotation}"/>
-            <child link="sonar_${suffix}"/>
-            <parent link="base_link"/>
+            <origin xyz="0 0 0.4" rpy="0 0 ${rotation}" />
+            <child link="sonar_${suffix}" />
+            <parent link="base_link" />
         </joint>
         <link name="sonar_${suffix}">
             <visual>
-                <origin xyz="0 0 0"/>
-                <geometry>
-                    <cylinder length="0.05" radius="0.05"/>
+                <origin xyz="0 0 0" />
+                <geometry>
+                    <cylinder length="0.05" radius="0.05" />
                 </geometry>
             </visual>
             <collision>
-                <origin xyz="0 0 0"/>
-                <geometry>
-                    <cylinder length="0.05" radius="0.05"/>
+                <origin xyz="0 0 0" />
+                <geometry>
+                    <cylinder length="0.05" radius="0.05" />
                 </geometry>
             </collision>
             <inertial>
-                <mass value="1"/>
-                <origin xyz="0 0 0"/>
+                <mass value="1" />
+                <origin xyz="0 0 0" />
                 <inertia
-                        ixx="1" ixy="0" ixz="0"
-                        iyy="1" iyz="0"
-                        izz="1"/>
+                    ixx="1" ixy="0" ixz="0"
+                    iyy="1" iyz="0"
+                    izz="1" />
             </inertial>
         </link>
@@ -173,57 +173,55 @@
         </gazebo>
     </xacro:macro>
-    <xacro:sonar_sensor suffix="0" rotation="-3.0"/>
-    <xacro:sonar_sensor suffix="1" rotation="-2.5"/>
-    <xacro:sonar_sensor suffix="2" rotation="-2.0"/>
-    <xacro:sonar_sensor suffix="3" rotation="-1.5"/>
-    <xacro:sonar_sensor suffix="4" rotation="-1.0"/>
-    <xacro:sonar_sensor suffix="5" rotation="-0.5"/>
-    <xacro:sonar_sensor suffix="6" rotation="0.0"/>
-    <xacro:sonar_sensor suffix="7" rotation="0.5"/>
-    <xacro:sonar_sensor suffix="8" rotation="1.0"/>
-    <xacro:sonar_sensor suffix="9" rotation="1.5"/>
-    <xacro:sonar_sensor suffix="10" rotation="2.0"/>
-    <xacro:sonar_sensor suffix="11" rotation="2.5"/>
-    <xacro:sonar_sensor suffix="12" rotation="3.0"/>
+    <xacro:sonar_sensor suffix="0" rotation="-3.0" />
+    <xacro:sonar_sensor suffix="1" rotation="-2.5" />
+    <xacro:sonar_sensor suffix="2" rotation="-2.0" />
+    <xacro:sonar_sensor suffix="3" rotation="-1.5" />
+    <xacro:sonar_sensor suffix="4" rotation="-1.0" />
+    <xacro:sonar_sensor suffix="5" rotation="-0.5" />
+    <xacro:sonar_sensor suffix="6" rotation="0.0" />
+    <xacro:sonar_sensor suffix="7" rotation="0.5" />
+    <xacro:sonar_sensor suffix="8" rotation="1.0" />
+    <xacro:sonar_sensor suffix="9" rotation="1.5" />
+    <xacro:sonar_sensor suffix="10" rotation="2.0" />
+    <xacro:sonar_sensor suffix="11" rotation="2.5" />
+    <xacro:sonar_sensor suffix="12" rotation="3.0" />
     <xacro:macro name="realsense_sensor" params="suffix tilt *origin">
         <joint name="realsense_joint_${suffix}" type="fixed">
-            <xacro:insert_block name="origin"/>
-            <child link="realsense_${suffix}"/>
-            <parent link="base_link"/>
-        </joint>
-        <link name="realsense_${suffix}">
-        </link>
+            <xacro:insert_block name="origin" />
+            <child link="realsense_${suffix}" />
+            <parent link="base_link" />
+        </joint>
+        <link name="realsense_${suffix}"></link>
         <joint name="realsense_joint_${suffix}_tilt" type="fixed">
-            <origin xyz="0 0 0" rpy="0 ${tilt} 0"/>
-            <child link="realsense_${suffix}_tilt"/>
-            <parent link="realsense_${suffix}"/>
-        </joint>
-        <link name="realsense_${suffix}_tilt">
-        </link>
+            <origin xyz="0 0 0" rpy="0 ${tilt} 0" />
+            <child link="realsense_${suffix}_tilt" />
+            <parent link="realsense_${suffix}" />
+        </joint>
+        <link name="realsense_${suffix}_tilt"></link>
         <joint name="realsense_${suffix}_camera_joint" type="fixed">
-            <origin xyz="0 0 0" rpy="${-pi/2} 0 ${-pi/2}"/>
-            <parent link="realsense_${suffix}_tilt"/>
-            <child link="realsense_${suffix}_camera"/>
+            <origin xyz="0 0 0" rpy="${-pi/2} 0 ${-pi/2}" />
+            <parent link="realsense_${suffix}_tilt" />
+            <child link="realsense_${suffix}_camera" />
         </joint>
         <link name="realsense_${suffix}_camera">
             <visual>
-                <origin xyz="0 0 0"/>
-                <geometry>
-                    <cylinder length="0.05" radius="0.01"/>
+                <origin xyz="0 0 0" />
+                <geometry>
+                    <cylinder length="0.05" radius="0.01" />
                 </geometry>
             </visual>
             <collision>
-                <origin xyz="0 0 0"/>
-                <geometry>
-                    <cylinder length="0.05" radius="0.01"/>
+                <origin xyz="0 0 0" />
+                <geometry>
+                    <cylinder length="0.05" radius="0.01" />
                 </geometry>
             </collision>
             <inertial>
-                <mass value="1"/>
-                <origin xyz="0 0 0"/>
+                <mass value="1" />
+                <origin xyz="0 0 0" />
                 <inertia
-                        ixx="1" ixy="0" ixz="0"
-                        iyy="1" iyz="0"
-                        izz="1"/>
+                    ixx="1" ixy="0" ixz="0"
+                    iyy="1" iyz="0"
+                    izz="1" />
             </inertial>
         </link>
@@ -240,6 +238,5 @@
                         <format>R8G8B8</format>
                     </image>
-                    <depth_camera>
-                    </depth_camera>
+                    <depth_camera></depth_camera>
                     <clip>
                         <near>0.1</near>
@@ -247,6 +244,5 @@
                     </clip>
                 </camera>
-                <depth_camera>
-                </depth_camera>
+                <depth_camera></depth_camera>
                 <plugin name="gazebo_depth_plugin" filename="libgazebo_depth_plugin.so">
                     <updateRate>4</updateRate>
@@ -257,14 +253,14 @@
     </xacro:macro>
     <xacro:realsense_sensor suffix="front" tilt="${-pi / 6}">
-        <origin xyz="0.4 0.0 1.0" rpy="${-pi / 2} ${pi / 2} ${-pi / 2}"/>
+        <origin xyz="0.4 0.0 1.0" rpy="${-pi / 2} ${pi / 2} ${-pi / 2}" />
     </xacro:realsense_sensor>
     <xacro:realsense_sensor suffix="back" tilt="${-pi / 6}">
-        <origin xyz="-0.4 0.0 1.0" rpy="${-pi / 2} ${pi / 2} ${pi / 2}"/>
+        <origin xyz="-0.4 0.0 1.0" rpy="${-pi / 2} ${pi / 2} ${pi / 2}" />
     </xacro:realsense_sensor>
     <xacro:realsense_sensor suffix="left" tilt="${-pi / 6}">
-        <origin xyz="0.0 0.4 1.0" rpy="${-pi / 2} ${pi / 2} 0"/>
+        <origin xyz="0.0 0.4 1.0" rpy="${-pi / 2} ${pi / 2} 0" />
     </xacro:realsense_sensor>
     <xacro:realsense_sensor suffix="right" tilt="${-pi / 6}">
-        <origin xyz="0.0 -0.4 1.0" rpy="${-pi / 2} ${pi / 2} ${pi}"/>
+        <origin xyz="0.0 -0.4 1.0" rpy="${-pi / 2} ${pi / 2} ${pi}" />
     </xacro:realsense_sensor>
     <!--<xacro:realsense_sensor suffix="back">-->

File: gridmap/test/robot.urdf.xacro (robot description, xacro)
@@ -18,22 +18,22 @@
     <link name="base_link">
         <visual>
-            <origin xyz="0 0 0.05"/>
-            <geometry>
-                <box size="0.5 0.5 0.1"/>
+            <origin xyz="0 0 0.05" />
+            <geometry>
+                <box size="0.5 0.5 0.1" />
             </geometry>
         </visual>
         <collision>
-            <origin xyz="0 0 0.05"/>
-            <geometry>
-                <box size="0.5 0.5 0.1"/>
+            <origin xyz="0 0 0.05" />
+            <geometry>
+                <box size="0.5 0.5 0.1" />
             </geometry>
         </collision>
         <inertial>
-            <origin xyz="0 0 0" rpy="0 0 0"/>
-            <mass value="1"/>
+            <origin xyz="0 0 0" rpy="0 0 0" />
+            <mass value="1" />
             <inertia
-                    ixx="1" ixy="0" ixz="0"
-                    iyy="1" iyz="0"
-                    izz="1"/>
+                ixx="1" ixy="0" ixz="0"
+                iyy="1" iyz="0"
+                izz="1" />
         </inertial>
     </link>
@@ -49,28 +49,28 @@
     <xacro:macro name="laser_sensor" params="suffix rotation">
         <joint name="laser_joint_${suffix}" type="fixed">
-            <origin xyz="0 0 0.4" rpy="0 0 ${rotation}"/>
-            <child link="laser_${suffix}"/>
-            <parent link="base_link"/>
+            <origin xyz="0 0 0.4" rpy="0 0 ${rotation}" />
+            <child link="laser_${suffix}" />
+            <parent link="base_link" />
         </joint>
         <link name="laser_${suffix}">
             <visual>
-                <origin xyz="0 0 0"/>
-                <geometry>
-                    <cylinder length="0.05" radius="0.05"/>
+                <origin xyz="0 0 0" />
+                <geometry>
+                    <cylinder length="0.05" radius="0.05" />
                 </geometry>
             </visual>
             <collision>
-                <origin xyz="0 0 0"/>
-                <geometry>
-                    <cylinder length="0.05" radius="0.05"/>
+                <origin xyz="0 0 0" />
+                <geometry>
+                    <cylinder length="0.05" radius="0.05" />
                 </geometry>
             </collision>
             <inertial>
-                <mass value="1"/>
-                <origin xyz="0 0 0"/>
+                <mass value="1" />
+                <origin xyz="0 0 0" />
                 <inertia
-                        ixx="1" ixy="0" ixz="0"
-                        iyy="1" iyz="0"
-                        izz="1"/>
+                    ixx="1" ixy="0" ixz="0"
+                    iyy="1" iyz="0"
+                    izz="1" />
             </inertial>
         </link>
@@ -107,32 +107,32 @@
         </gazebo>
     </xacro:macro>
-    <xacro:laser_sensor suffix="front" rotation="0.0"/>
-    <xacro:laser_sensor suffix="back" rotation="${pi}"/>
+    <xacro:laser_sensor suffix="front" rotation="0.0" />
+    <xacro:laser_sensor suffix="back" rotation="${pi}" />
     <xacro:macro name="sonar_sensor" params="suffix rotation">
         <joint name="sonar_${suffix}_joint" type="fixed">
-            <origin xyz="0 0 0.4" rpy="0 0 ${rotation}"/>
-            <child link="sonar_${suffix}"/>
-            <parent link="base_link"/>
+            <origin xyz="0 0 0.4" rpy="0 0 ${rotation}" />
+            <child link="sonar_${suffix}" />
+            <parent link="base_link" />
         </joint>
         <link name="sonar_${suffix}">
             <visual>
-                <origin xyz="0 0 0"/>
-                <geometry>
-                    <cylinder length="0.05" radius="0.05"/>
+                <origin xyz="0 0 0" />
+                <geometry>
+                    <cylinder length="0.05" radius="0.05" />
                 </geometry>
             </visual>
             <collision>
-                <origin xyz="0 0 0"/>
-                <geometry>
-                    <cylinder length="0.05" radius="0.05"/>
+                <origin xyz="0 0 0" />
+                <geometry>
+                    <cylinder length="0.05" radius="0.05" />
                 </geometry>
             </collision>
             <inertial>
-                <mass value="1"/>
-                <origin xyz="0 0 0"/>
+                <mass value="1" />
+                <origin xyz="0 0 0" />
                 <inertia
-                        ixx="1" ixy="0" ixz="0"
-                        iyy="1" iyz="0"
-                        izz="1"/>
+                    ixx="1" ixy="0" ixz="0"
+                    iyy="1" iyz="0"
+                    izz="1" />
             </inertial>
         </link>
@@ -184,7 +184,7 @@
     <!--<xacro:sonar_sensor suffix="12" rotation="3.0"/>-->
     <joint name="camera_joint" type="fixed">
-        <origin xyz="0.0 0.0 0.6" rpy="0.0 ${pi/2} 0.0"/>
-        <parent link="base_link"/>
-        <child link="camera"/>
+        <origin xyz="0.0 0.0 0.6" rpy="0.0 ${pi/2} 0.0" />
+        <parent link="base_link" />
+        <child link="camera" />
     </joint>
     <gazebo reference="camera_joint">
@@ -193,18 +193,18 @@
     <link name="camera">
         <inertial>
-            <mass value="1"/>
-            <inertia ixx="1e-6" ixy="0" ixz="0" iyy="1e-6" iyz="0" izz="1e-6"/>
+            <mass value="1" />
+            <inertia ixx="1e-6" ixy="0" ixz="0" iyy="1e-6" iyz="0" izz="1e-6" />
         </inertial>
         <visual>
-            <origin xyz="0 0 0.01" rpy="0 0 0"/>
-            <geometry>
-                <cylinder radius="0.016" length="0.080"/>
-            </geometry>
-            <material name="black"/>
+            <origin xyz="0 0 0.01" rpy="0 0 0" />
+            <geometry>
+                <cylinder radius="0.016" length="0.080" />
+            </geometry>
+            <material name="black" />
         </visual>
         <collision>
-            <origin xyz="0 0 0.01" rpy="0 0 0"/>
-            <geometry>
-                <cylinder radius="0.016" length="0.080"/>
+            <origin xyz="0 0 0.01" rpy="0 0 0" />
+            <geometry>
+                <cylinder radius="0.016" length="0.080" />
             </geometry>
         </collision>
